Commit message: Add robot model files, launch files, and Gazebo integration
- Added URDF and XACRO robot description files for obstacle_bot
- Added meshes for left and right wheels (STL files)
- Created Gazebo configuration file with physics and control plugins
- Added launch files for RViz display and Gazebo simulation
- Updated CMakeLists.txt to install model directory instead of urdf
- Updated display.launch.py to use model directory path
- Added xacro dependency to package.xml
- Updated .gitignore to exclude build artifacts
- Updated RViz configuration for better visualization

File: obstacle_bots_ws/src/obstacle_bot_cpp/model/obstacle_bot.urdf (robot description, URDF)
Before this commit: robot obstacle_bot, 4 links, 3 joints
Links:
- removed link Roda_L
- removed link Roda_R
- removed link world
- added link Caster_wheel, mass 0.01; collision sphere radius=0.008; visual sphere radius=0.008
- added link Left_wheel, mass 0.05; collision cylinder length=0.006 radius=0.017; visual cylinder length=0.006 radius=0.017
- added link Right_wheel, mass 0.05; collision cylinder length=0.006 radius=0.017; visual cylinder length=0.006 radius=0.017
- link Base: mass 0.158789661904281 -> 0.2; geometry collision box size=0.08 0.08 0.04; visual box size=0.08 0.08 0.04
Joints:
- removed joint Roda_L
- removed joint Roda_R
- removed joint world_to_base
- added joint Caster_wheel_joint: type fixed, parent Base, child Caster_wheel, origin xyz=0.03 0 0 rpy=0 0 0
- added joint Left_wheel_joint: type continuous, parent Base, child Left_wheel, origin xyz=0 0.0403 0.008 rpy=1.5708 0 0, axis 0 0 1
- added joint Right_wheel_joint: type continuous, parent Base, child Right_wheel, origin xyz=0 -0.0403 0.008 rpy=1.5708 0 0, axis 0 0 1
